File: hardware/motherboard/motherboard.kicad_sch (KiCad schematic)
At the start: 31 parts, among them J3 RFShield_TwoPieces, U1 TART Correlator Socket, U15 74LVC1G04SE-7, U2 CS48520S, X2 1XXB16368MBA

Commit message: Update to KiCAD 10
Parts:
- renumbered C1 to C22, C1 to C4, C1 to C5, TP2 to TP12, TP2 to TP13, TP2 to TP14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
