File: hardware/motherboard/motherboard.kicad_pcb (KiCad board)
At the start: 6 copper layers, 199.4 x 169 mm, 100 parts, among them J1 RADIO 1-4, J10 swd-connect-3, J14 9-28V, J2 RADIO 5-8, J3 RFShield_TwoPieces, J4 RADIO 1-4, J5 RADIO 5-8, J6 RADIO 1-4, J7 RADIO 5-8, J8 RADIO 1-4, J9 RADIO 5-8, SW1 Reset, U1 TART Correlator Socket, U10 LM2576SX-5.0, U11 SN74LV1T34DCK, U12 SN74LV1T34DCK, U13 SN74LV1T34DCK, U14 SN74LV1T34DCK, U15 74LVC1G04SE-7, U2 ch32v003f4u6, U3 AMS1117-3.3, U4 AMS1117-3.3, U5 AMS1117-3.3, U6 AMS1117-3.3, U7 AMS1117-3.3, U8 SN74LV1T34DCK, U9 CS48520S, X2 1XXB16368MBA

Commit message: add impedance matching resistors to RS485
Other:
- board text added: "TART Radio Telescope Version 26.08.0 (C) Tim Molteno (tim@elec.ac.nz) GPL v3.0, July 2026"
- board text removed: "TART Radio Telescope Version 3.0.0b3 (C) Tim Molteno (tim@elec.ac.nz) GPL v3.0, July 2024"
