File: hardware/spartan6_correlator/psu.kicad_sch (KiCad schematic)
At the start: 0 parts

Commit message: Added much more
Parts:
- added C1, C2: 4.7uF, symbol Device:C
- added C3, C4: 120pF, symbol Device:C
- added C5: 10uF, symbol Device:C
- added C6, C7: 22uF, symbol Device:C
- added L1, L2: 1 uH, symbol Device:L
- added R1, R4: 470k, symbol Device:R
- added R2: 450k, symbol Device:R
- added R3, R5, R6: 100k, symbol Device:R
- added U2, U5: TPS62A01DRL, Package_TO_SOT_SMD:SOT-563, symbol Regulator_Switching:TPS62A01DRL
Connections:
- new net: L2.1, U5.2 (SW)
- new net: L1.1, U2.2 (SW)
- new net: C4.2, R5.2, R6.1, U5.5 (FB)
- new net: R4.1, U5.6 (PG)
- new net: C3.2, R2.2, R3.1, U2.5 (FB)
- new net: R1.1, U2.6 (PG)
- new net +1V2: C4.1, C6.1, C7.1, L2.2, R4.2, R5.1
- new net +3V3: C2.1, C3.1, C5.1, L1.2, R1.2, R2.1, U5.3 (VIN), U5.4 (EN)
- new net +5V: C1.1, U2.3 (VIN), U2.4 (EN)
- new net GND: C1.2, C2.2, C5.2, C6.2, C7.2, R3.2, R6.2, U2.1 (GND), U5.1 (GND)
Other:
- note added: "Dual 3.3v AND 1.2V supply from 5V"
- note added: "R1 = R2 * (V_out / 0.6 - 1) = 100k (3.3 / 0.6 - 1) = 450k"
- note added: "R3 = R4 * (V_out / 0.6 - 1) = 100k (1.2 / 0.6 - 1) = 100k"

Commit message: Updates. Lots of them
Other:
- note added: "Should the PG pin of the 3.3V be used to enable the 1.2 V regulator?"
Changed lines of the file:
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@@
+		)
+	)
+	(text "Should the PG pin of the 3.3V be used to enable the 1.2 V regulator?"
+		(exclude_from_sim no)
+		(at 83.312 81.534 0)
+		(effects
+			(font
+				(size 1.27 1.27)
+			)
 		)
 	)

Commit message: Fix SDRAM to correct model
Parts:
- removed L1: 1 uH, symbol Device:L
- added L3: 1 uH, Inductor_SMD:L_1008_2520Metric, symbol Device:L
- C1, C2: footprint (none) -> Capacitor_SMD:C_0402_1005Metric; LCSC (none) -> C23733
- C3, C4, C5: footprint (none) -> Capacitor_SMD:C_0402_1005Metric
- C6, C7: footprint (none) -> Capacitor_SMD:C_0603_1608Metric; LCSC (none) -> C59461
- L2: footprint (none) -> Inductor_SMD:L_1008_2520Metric; LCSC (none) -> C5832370
- R1, R2, R3, R4, R5, R6: footprint (none) -> Resistor_SMD:R_0402_1005Metric
Connections:
- net +3V3: now also L3.2
- net at U2.2 (SW): now also L3.1

Commit message: Onto the board
Parts:
- removed R4: 470k, Resistor_SMD:R_0402_1005Metric, symbol Device:R
- added R10, R9: 0, Resistor_SMD:R_0402_1005Metric, symbol Device:R
Connections:
- net +3V3: now also R9.1; no longer U5.4 (EN)
- net 3V3_GOOD: now reaches R1.1, U2.6 (PG)
- net 3V3_GOOD: now also R10.2
- new net: R10.1, R9.2, U5.4 (EN)
- no-connect marks 0 -> 1
Other:
- moved on the sheet: C2

Commit message: Latest version
Parts:
- C3, C4: LCSC (none) -> C106996
- C5: LCSC (none) -> C15525
- R1: value 470k -> 453k; LCSC (none) -> C27009
- R10, R9: LCSC (none) -> C17168
- R2: value 450k -> 453k; LCSC (none) -> C27009
- R3, R5, R6: LCSC (none) -> C25741
Changed lines of the file:
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@@
+			)
+		)
+		(property "LCSC" "C17168"
+			(at 56.134 130.81 0)
+			(effects
+				(font
+					(size 1.27 1.27)
+				)
+				(hide yes)
 			)
 		)
@@
 			)
 		)
+		(property "LCSC" "C15525"
+			(at 111.76 55.8799 0)
+			(effects
+				(font
+					(size 1.27 1.27)
+				)
+				(hide yes)
+			)
+		)
 		(pin "2"
 		)
@@
 			)
 		)
+		(property "LCSC" "C25741"
+			(at 87.63 66.0399 0)
+			(effects
+				(font
+					(size 1.27 1.27)
+				)
+				(hide yes)
+			)
+		)
 		(pin "1"
 		)
@@
 			)
 		)
+		(property "LCSC" "C25741"
+			(at 87.63 142.2399 0)
+			(effects
+				(font
+					(size 1.27 1.27)
+				)
+				(hide yes)
+			)
+		)
 		(pin "1"
 		)
@@
 			)
 		)
-		(property "Value" "450k"
+		(property "Value" "453k"
 			(at 87.63 58.4199 0)
 			(effects
@@
 			)
 		)
+		(property "LCSC" "C27009"
+			(at 85.09 57.15 0)
+			(effects
+				(font
+					(size 1.27 1.27)
+				)
+				(hide yes)
+			)
+		)
 		(pin "1"
 		)
@@
 			)
 		)
+		(property "LCSC" "C17168"
+			(at 56.134 138.43 0)
+			(effects
+				(font
+					(size 1.27 1.27)
+				)
+				(hide yes)
+			)
+		)
 		(pin "1"
 		)
@@
 			)
 		)
+		(property "LCSC" "C106996"
+			(at 99.06 55.8799 0)
+			(effects
+				(font
+					(size 1.27 1.27)
+				)
+				(hide yes)
+			)
+		)
 		(pin "2"
 		)
@@
 			)
 		)
+		(property "LCSC" "C106996"
+			(at 99.06 132.0799 0)
+			(effects
+				(font
+					(size 1.27 1.27)
+				)
+				(hide yes)
+			)
+		)
 		(pin "2"
 		)
@@
 			)
 		)
-		(property "Value" "470k"
+		(property "Value" "453k"
 			(at 87.63 45.7199 0)
 			(effects
@@
 			)
 		)
+		(property "LCSC" "C27009"
+			(at 85.09 44.45 0)
+			(effects
+				(font
+					(size 1.27 1.27)
+				)
+				(hide yes)
+			)
+		)
 		(pin "1"
 		)
@@
 			(effects
 				(font
+					(size 1.27 1.27)
+				)
+				(hide yes)
+			)
+		)
+		(property "LCSC" "C25741"
+			(at 87.63 132.0799 0)
+			(effects
+				(font
