File: hardware/ufl_radio/ufl_radio.kicad_sch (KiCad schematic)
At the start: 26 parts, among them U2 CS48520S, U6 CDCV304PW

Commit message: Replace the RS485 driver as it is no longer in production
Parts:
- removed U2: CS48520S, Package_SO:SOIC-8_3.9x4.9mm_P1.27mm, symbol tart:CS48520S
- added U2: CS48520AS, Package_SO:SOIC-8_3.9x4.9mm_P1.27mm, symbol tart:CS48520AS
Connections:
- net CLKIN: now also U2.1 (RO)
- net GNDREF: now also U2.2 (REB), U2.5 (GND)
- net VCC: now also U2.8 (VCC)
- net at J1.A14 (REFCLK-): now also U2.6 (A)
- net at J1.A13 (REFCLK+): now also U2.7 (B)
Changed lines of the file:
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@@
-	)
-	(symbol
-		(lib_id "tart:CS48520S")
-		(at 193.04 57.15 0)
-		(unit 1)
-		(exclude_from_sim no)
-		(in_bom yes)
-		(on_board yes)
-		(dnp no)
-		(property "Reference" "U2"
-			(at 191.77 57.15 0)
-			(effects
-				(font
-					(size 1.27 1.27)
-				)
-				(justify left)
-			)
-		)
-		(property "Value" "CS48520S"
-			(at 194.9959 44.45 0)
-			(effects
-				(font
-					(size 1.27 1.27)
-				)
-				(justify left)
-			)
-		)
-		(property "Footprint" "Package_SO:SOIC-8_3.9x4.9mm_P1.27mm"
-			(at 193.04 57.15 0)
-			(effects
-				(font
-					(size 1.27 1.27)
-				)
-				(hide yes)
-			)
-		)
-		(property "Datasheet" "http://e.chipanalog.com/product/cs48520s/"
-			(at 193.04 57.15 0)
-			(effects
-				(font
-					(size 1.27 1.27)
-				)
-				(hide yes)
-			)
-		)
-		(property "Description" "The CS485xx family of devices are low-power half-duplex transceivers for RS-485/RS-422 communications"
-			(at 193.04 57.15 0)
-			(effects
-				(font
-					(size 1.27 1.27)
-				)
-				(hide yes)
-			)
-		)
-		(property "LCSC" "C5184817"
-			(at 194.9959 46.99 0)
-			(effects
-				(font
-					(size 1.27 1.27)
-				)
-				(justify left)
-			)
-		)
-		(pin "1"
-		)
-		(pin "2"
-		)
-		(pin "3"
-		)
-		(pin "4"
-		)
-		(pin "5"
-		)
-		(pin "6"
-		)
-		(pin "7"
-		)
-		(pin "8"
-		)
-		(instances
-			(project "design"
-				(path "/6dbd6c42-edf6-461d-b7ca-066e49b0019c"
-					(reference "U2")
-					(unit 1)
-				)
-			)
-		)
 	)
 	(symbol
@@
 					(unit 1)
 				)
+			)
+		)
+	)
+	(symbol
+		(lib_id "tart:CS48520AS")
+		(at 193.04 57.15 0)
+		(unit 1)
+		(exclude_from_sim no)
+		(in_bom yes)
+		(on_board yes)
+		(dnp no)
+		(fields_autoplaced yes)
+		(property "Reference" "U2"
+			(at 195.1833 40.64 0)
+			(effects
+				(font
+					(size 1.27 1.27)
+				)
+				(justify left)
+			)
+		)
+		(property "Value" "CS48520AS"
+			(at 195.1833 43.18 0)
+			(effects
+				(font
+					(size 1.27 1.27)
+				)
+				(justify left)
+			)
+		)
+		(property "Footprint" "Package_SO:SOIC-8_3.9x4.9mm_P1.27mm"
+			(at 191.77 72.39 0)
+			(effects
+				(font
+					(size 1.27 1.27)
+				)
+				(hide yes)
+			)
+		)
+		(property "Datasheet" "http://e.chipanalog.com/product/cs48520s/"
+			(at 193.04 57.15 0)
+			(effects
+				(font
+					(size 1.27 1.27)
+				)
+				(hide yes)
+			)
+		)
+		(property "Description" "The CS485xx family of devices are low-power half-duplex transceivers for RS-485/RS-422 communications"
+			(at 193.04 57.15 0)
+			(effects
+				(font
+					(size 1.27 1.27)
+				)
+				(hide yes)
+			)
+		)
+		(property "LCSC" "C7422554"
+			(at 195.1833 45.72 0)
+			(effects
+				(font
+					(size 1.27 1.27)
+				)
+				(justify left)
+			)
+		)
+		(pin "6"
+		)
+		(pin "3"
+		)
+		(pin "2"
+		)
+		(pin "1"
+		)
+		(pin "8"
+		)
+		(pin "5"
+		)
+		(pin "4"
+		)
+		(pin "7"
+		)
+		(instances
+			(project ""
+				(path "/6dbd6c42-edf6-461d-b7ca-066e49b0019c"
+					(reference "U2")
+					(unit 1)
+				)

Commit message: Update to new DFN8 package
Parts:
- removed U2: CS48520AS, Package_SO:SOIC-8_3.9x4.9mm_P1.27mm, symbol tart:CS48520AS
- added U2: CS48520AD, Package_DFN_QFN:DFN-8-1EP_3x3mm_P0.65mm_EP1.6x2.56mm, symbol tart:CS48520AD
Connections:
- net CLKIN: now also U2.1 (RO)
- net GNDREF: now also U2.2 (REB), U2.5 (GND), U2.9 (GND)
- net VCC: now also U2.8 (VCC)
- net at J1.A13 (REFCLK+): now also U2.7 (B)
- net at J1.A14 (REFCLK-): now also U2.6 (A)
Changed lines of the file:
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@@
 	)
 	(junction
+		(at 189.23 68.58)
+		(diameter 0)
+		(color 0 0 0 0)
+	)
+	(junction
 		(at 242.57 73.66)
 		(diameter 0)
@@
 	(wire
 		(pts
+			(xy 189.23 68.58) (xy 193.04 68.58)
+		)
+		(stroke
+			(width 0)
+			(type default)
+		)
+	)
+	(wire
+		(pts
 			(xy 137.16 78.74) (xy 140.97 78.74)
 		)
@@
 	(wire
 		(pts
-			(xy 179.07 68.58) (xy 193.04 68.58)
+			(xy 179.07 68.58) (xy 189.23 68.58)
 		)
 		(stroke
@@
 	)
 	(symbol
+		(lib_id "tart:CS48520AD")
+		(at 193.04 57.15 0)
+		(unit 1)
+		(exclude_from_sim no)
+		(in_bom yes)
+		(on_board yes)
+		(dnp no)
+		(fields_autoplaced yes)
+		(property "Reference" "U2"
+			(at 195.1833 40.64 0)
+			(effects
+				(font
+					(size 1.27 1.27)
+				)
+				(justify left)
+			)
+		)
+		(property "Value" "CS48520AD"
+			(at 195.1833 43.18 0)
+			(effects
+				(font
+					(size 1.27 1.27)
+				)
+				(justify left)
+			)
+		)
+		(property "Footprint" "Package_DFN_QFN:DFN-8-1EP_3x3mm_P0.65mm_EP1.6x2.56mm"
+			(at 191.77 72.39 0)
+			(effects
+				(font
+					(size 1.27 1.27)
+				)
+				(hide yes)
+			)
+		)
+		(property "Datasheet" "http://e.chipanalog.com/product/cs48520s/"
+			(at 193.04 57.15 0)
+			(effects
+				(font
+					(size 1.27 1.27)
+				)
+				(hide yes)
+			)
+		)
+		(property "Description" "The CS485xx family of devices are low-power half-duplex transceivers for RS-485/RS-422 communications"
+			(at 193.04 57.15 0)
+			(effects
+				(font
+					(size 1.27 1.27)
+				)
+				(hide yes)
+			)
+		)
+		(property "LCSC" "C7422569"
+			(at 195.1833 45.72 0)
+			(effects
+				(font
+					(size 1.27 1.27)
+				)
+				(justify left)
+			)
+		)
+		(pin "6"
+		)
+		(pin "9"
+		)
+		(pin "3"
+		)
+		(pin "8"
+		)
+		(pin "5"
+		)
+		(pin "2"
+		)
+		(pin "1"
+		)
+		(pin "7"
+		)
+		(pin "4"
+		)
+		(instances
+			(project ""
+				(path "/6dbd6c42-edf6-461d-b7ca-066e49b0019c"
+					(reference "U2")
+					(unit 1)
+				)
+			)
+		)
+	)
+	(symbol
 		(lib_id "power:GNDREF")
 		(at 193.04 69.85 0)
@@
 					(unit 1)
 				)
-			)
-		)
-	)
-	(symbol
-		(lib_id "tart:CS48520AS")
-		(at 193.04 57.15 0)
-		(unit 1)
-		(exclude_from_sim no)
-		(in_bom yes)
-		(on_board yes)
-		(dnp no)
-		(fields_autoplaced yes)
-		(property "Reference" "U2"
-			(at 195.1833 40.64 0)
-			(effects
-				(font
-					(size 1.27 1.27)
-				)
-				(justify left)
-			)
-		)
-		(property "Value" "CS48520AS"
-			(at 195.1833 43.18 0)
-			(effects
-				(font
-					(size 1.27 1.27)
-				)
-				(justify left)
-			)
-		)
-		(property "Footprint" "Package_SO:SOIC-8_3.9x4.9mm_P1.27mm"
-			(at 191.77 72.39 0)
-			(effects
-				(font
-					(size 1.27 1.27)
-				)
-				(hide yes)
-			)
-		)
-		(property "Datasheet" "http://e.chipanalog.com/product/cs48520s/"
-			(at 193.04 57.15 0)
-			(effects
-				(font
-					(size 1.27 1.27)
-				)
-				(hide yes)
-			)
-		)
-		(property "Description" "The CS485xx family of devices are low-power half-duplex transceivers for RS-485/RS-422 communications"
-			(at 193.04 57.15 0)
-			(effects
-				(font
-					(size 1.27 1.27)
-				)
-				(hide yes)
-			)
-		)
-		(property "LCSC" "C7422554"
-			(at 195.1833 45.72 0)
-			(effects
-				(font
-					(size 1.27 1.27)
-				)
-				(justify left)
-			)
-		)
-		(pin "6"
-		)
-		(pin "3"
-		)
-		(pin "2"
-		)
-		(pin "1"
-		)
-		(pin "8"
-		)
-		(pin "5"
-		)
-		(pin "4"
-		)
-		(pin "7"
-		)
-		(instances
-			(project ""
-				(path "/6dbd6c42-edf6-461d-b7ca-066e49b0019c"
-					(reference "U2")
-					(unit 1)
-				)

Commit message: Update to KiCAD 10
Parts:
- J1: value ~ -> (none)
